File: left.sch (KiCad schematic (older format))
At the start: 57 parts, among them J1 Speaker, J3 ISP, J7 WS2812>, P2 UJ2-MBH-1-SMT, P3 >WS2812, P4 SJ-43514-SMT, SW1 Socket, SW10 Socket, SW11 Socket, SW12 Socket, SW13 Socket, SW14 Socket, SW15 Socket, SW16 Socket, SW17 Socket, SW18 Socket, SW19 Socket, SW2 Socket, SW20 Socket, SW21 Socket, SW22 Socket, SW23 Socket, SW24 Socket, SW3 Socket, SW4 Socket, SW5 Socket, SW6 Socket, SW7 Socket, SW8 Socket, SW9 Socket, U1 ATMega32U4, Y1 16MHz

Commit message: renamed files, and generated xy files
Parts:
- SW24: value Socket -> Socket-overlap
Changed lines of the file:
@@
 P 10350 4825
 F 0 "SW24" H 10350 5110 50  0000 C CNN
-F 1 "Socket" H 10350 5019 50  0000 C CNN
+F 1 "Socket-overlap" H 10350 5019 50  0000 C CNN
 F 2 "CherryMX:Kailh-socket" H 10350 5025 50  0001 C CNN
 F 3 "" H 10350 5025 50  0001 C CNN
@@
 	1975 4775 2600 4775
 $Comp
-L lets_split_panel-rescue:VCC-RESCUE-lets_split_panel #PWR?
+L lets_split_panel-rescue:VCC-RESCUE-lets_split_panel #PWR06
 U 1 1 5B50839C
 P 1900 7150
-F 0 "#PWR?" H 1900 7000 50  0001 C CNN
+F 0 "#PWR06" H 1900 7000 50  0001 C CNN
 F 1 "VCC" H 1900 7300 50  0000 C CNN
 F 2 "" H 1900 7150 50  0000 C CNN

Commit message: Added BOM and 3D file
Parts:
- C1, C2, C3, C4: symbol lets_split_panel-rescue:C_Small-RESCUE-lets_split_panel -> vitamins_included-rescue:C_Small-RESCUE-lets_split_panel-lets_split_panel-rescue
- J1: symbol lets_split_panel-rescue:Conn_01x02-RESCUE-lets_split_panel -> vitamins_included-rescue:Conn_01x02-RESCUE-lets_split_panel-lets_split_panel-rescue
- J3: symbol lets_split_panel-rescue:Conn_02x03_Odd_Even-RESCUE-lets_split_panel -> vitamins_included-rescue:Conn_02x03_Odd_Even-RESCUE-lets_split_panel-lets_split_panel-rescue
- J7: symbol lets_split_panel-rescue:Conn_01x01-RESCUE-lets_split_panel -> vitamins_included-rescue:Conn_01x01-RESCUE-lets_split_panel-lets_split_panel-rescue
- JP1, JP2: symbol lets_split_panel-rescue:Jumper-RESCUE-lets_split_panel -> vitamins_included-rescue:Jumper-RESCUE-lets_split_panel-lets_split_panel-rescue
- P2: symbol lets_split_panel-rescue:USB_OTG-RESCUE-lets_split-RESCUE-lets_split_panel -> vitamins_included-rescue:USB_OTG-RESCUE-lets_split-RESCUE-lets_split_panel-lets_split_panel-rescue
- P3: symbol lets_split_panel-rescue:Conn_01x03-RESCUE-lets_split_panel -> vitamins_included-rescue:Conn_01x03-RESCUE-lets_split_panel-lets_split_panel-rescue
- P4: symbol lets_split_panel-rescue:Conn_01x04-RESCUE-lets_split_panel -> vitamins_included-rescue:Conn_01x04-RESCUE-lets_split_panel-lets_split_panel-rescue
- R1, R2, R3, R4, R5, R6: symbol lets_split_panel-rescue:R_Small-RESCUE-lets_split_panel -> vitamins_included-rescue:R_Small-RESCUE-lets_split_panel-lets_split_panel-rescue
- SW1, SW10, SW11, SW12, SW13, SW14, SW15, SW16, SW17, SW18, SW19, SW2, SW20, SW21, SW22, SW23, SW24, SW3, SW4, SW5, SW6, SW7, SW8, SW9: symbol lets_split_panel-rescue:SW_Push-RESCUE-lets_split_panel -> vitamins_included-rescue:SW_Push-RESCUE-lets_split_panel-lets_split_panel-rescue
- U1: symbol lets_split_panel-rescue:ATMega32U4-RESCUE-lets_split_panel -> vitamins_included-rescue:ATMega32U4-RESCUE-lets_split_panel-lets_split_panel-rescue
- Y1: symbol lets_split_panel-rescue:Crystal-RESCUE-lets_split_panel -> vitamins_included-rescue:Crystal-RESCUE-lets_split_panel-lets_split_panel-rescue

Commit message: Added resistors to allow MCU to determin which half it is on
Parts:
- added J2: reset, Connector_PinHeader_2.54mm:PinHeader_1x02_P2.54mm_Vertical, symbol Connector_Generic:Conn_01x02
- added R11: 4k7, Resistor_SMD:R_0603_1608Metric, symbol vitamins_included-rescue:R_Small-RESCUE-lets_split_panel-lets_split_panel-rescue
- R1, R2, R3, R4, R5, R6: footprint Resistors_SMD:R_0603 -> Resistor_SMD:R_0603_1608Metric
- SW1, SW10, SW11, SW12, SW13, SW14, SW15, SW16, SW17, SW18, SW19, SW2, SW20, SW21, SW22, SW23, SW24, SW3, SW4, SW5, SW6, SW7, SW8, SW9: footprint CherryMX:Kailh-socket -> sockets:Kailh-socket
Connections:
- wire segments 183 -> 188

Commit message: Changed to USB-C connector
Parts:
- removed P2: UJ2-MBH-1-SMT, Connectors:USB-Mini-B-SMD, symbol vitamins_included-rescue:USB_OTG-RESCUE-lets_split-RESCUE-lets_split_panel-lets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
- added J9: 12401598E4#2A, Connector_USB:USB_C_Receptacle_Amphenol_12401610E4-2A, symbol Connector:USB_C_Receptacle
- R3: value 200R -> 220R
Connections:
- wire segments 188 -> 205

Commit message: Added resistors to allow the firmware to determine version
Parts:
- added R13: 4k7, Resistor_SMD:R_0603_1608Metric, symbol vitamins_included-rescue:R_Small-RESCUE-lets_split_panel-lets_split_panel-rescue
- SW24: value Socket-overlap -> Socket
Connections:
- wire segments 205 -> 208
Changed lines of the file:
@@
 P 10750 3250
 F 0 "SW24" H 10750 3535 50  0000 C CNN
-F 1 "Socket-overlap" H 10750 3444 50  0000 C CNN
+F 1 "Socket" H 10750 3444 50  0000 C CNN
 F 2 "sockets:Kailh-socket" H 10750 3450 50  0001 C CNN
 F 3 "" H 10750 3450 50  0001 C CNN
@@
 	1    0    0    -1
 $EndComp
-Wire Wire Line
-	5725 4400 5725 4450
 $Comp
 L vitamins_included-rescue:GND-RESCUE-lets_split_panel-lets_split_panel-rescue #PWR024
 U 1 1 5B57FD0A
-P 5725 4450
-F 0 "#PWR024" H 5725 4200 50  0001 C CNN
-F 1 "GND" H 5725 4300 50  0000 C CNN
-F 2 "" H 5725 4450 50  0000 C CNN
-F 3 "" H 5725 4450 50  0000 C CNN
-	1    5725 4450
+P 5725 4575
+F 0 "#PWR024" H 5725 4325 50  0001 C CNN
+F 1 "GND" H 5725 4425 50  0000 C CNN
+F 2 "" H 5725 4575 50  0000 C CNN
+F 3 "" H 5725 4575 50  0000 C CNN
+	1    5725 4575
 	1    0    0    -1
 $EndComp
@@
 U 1 1 5B59BDE8
 P 5575 4400
-F 0 "R11" H 5605 4420 50  0000 L CNN
-F 1 "4k7" H 5605 4360 50  0000 L CNN
+F 0 "R11" H 5600 4425 50  0000 L CNN
+F 1 "4k7" H 5600 4350 50  0000 L CNN
 F 2 "Resistor_SMD:R_0603_1608Metric" H 5575 4400 50  0001 C CNN
 F 3 "" H 5575 4400 50  0000 C CNN
@@
 Wire Wire Line
 	925  7150 1025 7150
+Wire Wire Line
+	5175 4500 5475 4500
+$Comp
+L vitamins_included-rescue:R_Small-RESCUE-lets_split_panel-lets_split_panel-rescue R13
+U 1 1 5B569B84
+P 5575 4500
+F 0 "R13" H 5425 4525 50  0000 L CNN
+F 1 "4k7" H 5400 4450 50  0000 L CNN
+F 2 "Resistor_SMD:R_0603_1608Metric" H 5575 4500 50  0001 C CNN
+F 3 "" H 5575 4500 50  0000 C CNN
+	1    5575 4500
+	0    -1   -1   0
+$EndComp
+Wire Wire Line
+	5725 4400 5725 4500
+Wire Wire Line
+	5675 4500 5725 4500
+Connection ~ 5725 4500
+Wire Wire Line
+	5725 4500 5725 4575
 $EndSCHEMATC

Commit message: changed to rounded passive footprints
Parts:
- C1, C2, C3, C4: footprint Capacitors_SMD:C_0603 -> Capacitor_SMD:C_0603_1608Metric
- R11, R13: value 4k7 -> 220R
Changed lines of the file:
@@
 F 0 "C4" H 3517 6196 50  0000 L CNN
 F 1 "1uF" H 3517 6105 50  0000 L CNN
-F 2 "Capacitors_SMD:C_0603" H 3425 6150 50  0001 C CNN
+F 2 "Capacitor_SMD:C_0603_1608Metric" H 3425 6150 50  0001 C CNN
 F 3 "" H 3425 6150 50  0001 C CNN
 	1    3425 6150
@@
 F 0 "C2" V 3250 5500 50  0000 C CNN
 F 1 "18pF" V 3225 5300 50  0000 C CNN
-F 2 "Capacitors_SMD:C_0603" H 3325 5400 50  0001 C CNN
+F 2 "Capacitor_SMD:C_0603_1608Metric" H 3325 5400 50  0001 C CNN
 F 3 "" H 3325 5400 50  0001 C CNN
 	1    3325 5400
@@
 F 0 "C3" V 3500 5800 50  0000 C CNN
 F 1 "18pF" V 3425 5800 50  0000 C CNN
-F 2 "Capacitors_SMD:C_0603" H 3325 5800 50  0001 C CNN
+F 2 "Capacitor_SMD:C_0603_1608Metric" H 3325 5800 50  0001 C CNN
 F 3 "" H 3325 5800 50  0001 C CNN
 	1    3325 5800
@@
 F 0 "C1" H 2967 6721 50  0000 L CNN
 F 1 "1uF" H 2967 6630 50  0000 L CNN
-F 2 "Capacitors_SMD:C_0603" H 2875 6675 50  0001 C CNN
+F 2 "Capacitor_SMD:C_0603_1608Metric" H 2875 6675 50  0001 C CNN
 F 3 "" H 2875 6675 50  0001 C CNN
 	1    2875 6675
@@
 P 5575 4400
 F 0 "R11" H 5600 4425 50  0000 L CNN
-F 1 "4k7" H 5600 4350 50  0000 L CNN
+F 1 "220R" H 5600 4350 50  0000 L CNN
 F 2 "Resistor_SMD:R_0603_1608Metric" H 5575 4400 50  0001 C CNN
 F 3 "" H 5575 4400 50  0000 C CNN
@@
 U 1 1 5B569B84
 P 5575 4500
-F 0 "R13" H 5425 4525 50  0000 L CNN
-F 1 "4k7" H 5400 4450 50  0000 L CNN
+F 0 "R13" H 5375 4525 50  0000 L CNN
+F 1 "220R" H 5350 4450 50  0000 L CNN
 F 2 "Resistor_SMD:R_0603_1608Metric" H 5575 4500 50  0001 C CNN
 F 3 "" H 5575 4500 50  0000 C CNN

Commit message: Switched to connectors
Parts:
- J7: value WS2812> -> Sig
- J9: value 12401598E4#2A -> UTC16-G; footprint Connector_USB:USB_C_Receptacle_Amphenol_12401610E4-2A -> Connector_USB:USB_C_Receptacle_Palconn_UTC16-G
- P3: value >WS2812 -> WS2812
Changed lines of the file:
@@
 AR Path="/5A0DE9BD/59DDE6F8" Ref="P3"  Part="1"
 F 0 "P3" H 1650 1475 50  0000 C CNN
-F 1 ">WS2812" V 1750 1275 50  0000 C CNN
+F 1 "WS2812" V 1750 1275 50  0000 C CNN
 F 2 "Wirepads:SMD_PAD_1x03_Pitch2.54mm" H 1650 1275 50  0001 C CNN
 F 3 "" H 1650 1275 50  0000 C CNN
@@
 P 2100 1275
 F 0 "J7" H 2020 1050 50  0000 C CNN
-F 1 "WS2812>" H 2020 1141 50  0000 C CNN
+F 1 "Sig" H 2020 1141 50  0000 C CNN
 F 2 "Pin_Headers:Pin_Header_Straight_1x01_Pitch2.54mm" H 2100 1275 50  0001 C CNN
 F 3 "~" H 2100 1275 50  0001 C CNN
@@
 P 1125 5500
 F 0 "J9" H 1230 7067 50  0000 C CNN
-F 1 " 12401598E4#2A " H 1230 6976 50  0000 C CNN
-F 2 "Connector_USB:USB_C_Receptacle_Amphenol_12401610E4-2A" H 1275 5500 50  0001 C CNN
+F 1 "UTC16-G" H 1230 6976 50  0000 C CNN
+F 2 "Connector_USB:USB_C_Receptacle_Palconn_UTC16-G" H 1275 5500 50  0001 C CNN
 F 3 "http://www.usb.org/developers/docs/usb_31_033017.zip" H 1275 5500 50  0001 C CNN
 	1    1125 5500

Commit message: Added reset button, led, 3D models
Parts:
- added D27: red, LED_SMD:LED_0603_1608Metric_Castellated, symbol Device:LED_Small
- added R15: 220R, Resistor_SMD:R_0603_1608Metric, symbol vitamins_included-rescue:R_Small-RESCUE-lets_split_panel-lets_split_panel-rescue
- added SW49: FSMSM, Button_Switch_SMD:SW_SPST_FSMSM, symbol Switch:SW_SPST
Connections:
- wire segments 208 -> 220
Changed lines of the file:
@@
 L vitamins_included-rescue:Conn_02x03_Odd_Even-RESCUE-lets_split_panel-lets_split_panel-rescue J3
 U 1 1 5A10645D
-P 10275 5825
-F 0 "J3" H 10325 6142 50  0000 C CNN
-F 1 "ISP" H 10325 6051 50  0000 C CNN
-F 2 "Connector:Tag-Connect_TC2030-IDC-NL_2x03_P1.27mm_Vertical" H 10275 5825 50  0001 C CNN
-F 3 "" H 10275 5825 50  0001 C CNN
-	1    10275 5825
+P 4125 2525
+F 0 "J3" H 4175 2842 50  0000 C CNN
+F 1 "ISP" H 4175 2751 50  0000 C CNN
+F 2 "Connector:Tag-Connect_TC2030-IDC-NL_2x03_P1.27mm_Vertical" H 4125 2525 50  0001 C CNN
+F 3 "" H 4125 2525 50  0001 C CNN
+	1    4125 2525
 	1    0    0    -1
 $EndComp
@@
 L vitamins_included-rescue:VCC-RESCUE-lets_split_panel-lets_split_panel-rescue #PWR018
 U 1 1 5A10B959
-P 10625 5675
-F 0 "#PWR018" H 10625 5525 50  0001 C CNN
-F 1 "VCC" H 10625 5825 50  0000 C CNN
-F 2 "" H 10625 5675 50  0000 C CNN
-F 3 "" H 10625 5675 50  0000 C CNN
-	1    10625 5675
+P 4475 2375
+F 0 "#PWR018" H 4475 2225 50  0001 C CNN
+F 1 "VCC" H 4475 2525 50  0000 C CNN
+F 2 "" H 4475 2375 50  0000 C CNN
+F 3 "" H 4475 2375 50  0000 C CNN
+	1    4475 2375
 	1    0    0    -1
 $EndComp
@@
 L vitamins_included-rescue:GND-RESCUE-lets_split_panel-lets_split_panel-rescue #PWR019
 U 1 1 5A10BE44
-P 10625 5975
-F 0 "#PWR019" H 10625 5725 50  0001 C CNN
-F 1 "GND" H 10625 5825 50  0000 C CNN
-F 2 "" H 10625 5975 50  0000 C CNN
-F 3 "" H 10625 5975 50  0000 C CNN
-	1    10625 5975
+P 4475 2675
+F 0 "#PWR019" H 4475 2425 50  0001 C CNN
+F 1 "GND" H 4475 2525 50  0000 C CNN
+F 2 "" H 4475 2675 50  0000 C CNN
+F 3 "" H 4475 2675 50  0000 C CNN
+	1    4475 2675
 	1    0    0    -1
 $EndComp
@@
 	5175 4100 5250 4100
 Wire Wire Line
-	10625 5725 10625 5675
-Wire Wire Line
-	10575 5725 10625 5725
-Wire Wire Line
-	10625 5925 10625 5975
-Wire Wire Line
-	10575 5925 10625 5925
+	4475 2425 4475 2375
+Wire Wire Line
+	4425 2425 4475 2425
+Wire Wire Line
+	4475 2625 4475 2675
+Wire Wire Line
+	4425 2625 4475 2625
 Connection ~ 3575 900
 Wire Wire Line
@@
 Wire Wire Line
 	2825 4200 2825 4225
-Connection ~ 2825 4450
 Wire Wire Line
 	2825 4450 2825 4425
@@
 SCK
 Wire Wire Line
-	10025 5725 10075 5725
-Wire Wire Line
-	10575 5825 10625 5825
-Wire Wire Line
-	10075 5825 10025 5825
-Text Label 10025 5725 2    60   ~ 0
+	3875 2425 3925 2425
+Wire Wire Line
+	4425 2525 4475 2525
+Wire Wire Line
+	3925 2525 3875 2525
+Text Label 3875 2425 2    60   ~ 0
 MISO
-Text Label 10625 5825 0    60   ~ 0
+Text Label 4475 2525 0    60   ~ 0
 MOSI
-Text Label 10025 5825 2    60   ~ 0
+Text Label 3875 2525 2    60   ~ 0
 SCK
 Text Label 6200 3500 2    60   ~ 0
@@
 col5
 Wire Wire Line
-	10075 5925 10025 5925
-Text Label 10025 5925 2    60   ~ 0
+	3925 2625 3875 2625
+Text Label 3875 2625 2    60   ~ 0
 ~Reset
 Text Label 3325 4450 2    60   ~ 0
@@
 Connection ~ 11000 1300
 Wire Wire Line
-	2675 4450 2825 4450
-Wire Wire Line
 	3575 900  3625 900
 Wire Wire Line
@@
 L Connector_Generic:Conn_01x02 J2
 U 1 1 5B51F3C1
-P 2475 4450
-F 0 "J2" H 2555 4442 50  0000 L CNN
-F 1 "reset" H 2555 4351 50  0000 L CNN
-F 2 "Connector_PinHeader_2.54mm:PinHeader_1x02_P2.54mm_Vertical" H 2475 4450 50  0001 C CNN
-F 3 "~" H 2475 4450 50  0001 C CNN
-	1    2475 4450
+P 2125 2300
+F 0 "J2" H 2205 2292 50  0000 L CNN
+F 1 "reset" H 2205 2201 50  0000 L CNN
+F 2 "Connector_PinHeader_2.54mm:PinHeader_1x02_P2.54mm_Vertical" H 2125 2300 50  0001 C CNN
+F 3 "~" H 2125 2300 50  0001 C CNN
+	1    2125 2300
 	-1   0    0    -1
 $EndComp
-Wire Wire Line
-	2675 4550 2725 4550
-Wire Wire Line
-	2725 4550 2725 4600
 $Comp
 L vitamins_included-rescue:GND-RESCUE-lets_split_panel-lets_split_panel-rescue #PWR015
 U 1 1 5B531998
-P 2725 4600
-F 0 "#PWR015" H 2725 4350 50  0001 C CNN
-F 1 "GND" H 2725 4450 50  0000 C CNN
-F 2 "" H 2725 4600 50  0000 C CNN
-F 3 "" H 2725 4600 50  0000 C CNN
-	1    2725 4600
+P 2375 2650
+F 0 "#PWR015" H 2375 2400 50  0001 C CNN
+F 1 "GND" H 2375 2500 50  0000 C CNN
+F 2 "" H 2375 2650 50  0000 C CNN
+F 3 "" H 2375 2650 50  0000 C CNN
+	1    2375 2650
 	1    0    0    -1
 $EndComp
@@
 Wire Wire Line
 	5725 4500 5725 4575
+$Comp
+L Switch:SW_SPST SW49
+U 1 1 5B5C5906
+P 2425 2350
+F 0 "SW49" V 2379 2448 50  0000 L CNN
+F 1 "FSMSM" V 2470 2448 50  0000 L CNN
+F 2 "Button_Switch_SMD:SW_SPST_FSMSM" H 2425 2350 50  0001 C CNN
+F 3 "" H 2425 2350 50  0001 C CNN
+	1    2425 2350
+	0    1    1    0
+$EndComp
+Wire Wire Line
+	2325 2300 2375 2300
+Wire Wire Line
+	2375 2300 2375 2100
+Wire Wire Line
+	2375 2100 2425 2100
+Wire Wire Line
+	2425 2100 2425 2150
+Wire Wire Line
+	2325 2400 2375 2400
+Wire Wire Line
+	2375 2600 2425 2600
+Wire Wire Line
+	2425 2600 2425 2550
+Wire Wire Line
+	2375 2400 2375 2600
+Connection ~ 2375 2600
+Wire Wire Line
+	2375 2600 2375 2650
+Wire Wire Line
+	2375 2100 2375 2025
+Connection ~ 2375 2100
+Text Label 2375 2025 3    60   ~ 0
+~Reset
+$Comp
+L Device:LED_Small D27
+U 1 1 5B5D7908
+P 5350 5500
+F 0 "D27" H 5350 5295 50  0000 C CNN
+F 1 "red" H 5350 5386 50  0000 C CNN
+F 2 "LED_SMD:LED_0603_1608Metric_Castellated" V 5350 5500 50  0001 C CNN
+F 3 "~" V 5350 5500 50  0001 C CNN
+	1    5350 5500
+	-1   0    0    1
+$EndComp
+Wire Wire Line
+	5175 5600 5225 5600
+Wire Wire Line
+	5225 5600 5225 5500
+Wire Wire Line
+	5225 5500 5250 5500
+$Comp
+L vitamins_included-rescue:R_Small-RESCUE-lets_split_panel-lets_split_panel-rescue R15
+U 1 1 5B5E58FB
+P 5550 5500
+F 0 "R15" H 5575 5525 50  0000 L CNN
+F 1 "220R" H 5575 5450 50  0000 L CNN
+F 2 "Resistor_SMD:R_0603_1608Metric" H 5550 5500 50  0001 C CNN
+F 3 "" H 5550 5500 50  0000 C CNN
+	1    5550 5500
+	0    -1   -1   0
+$EndComp
+Wire Wire Line
+	5650 5500 5700 5500
+Wire Wire Line
+	5700 5500 5700 5550
+$Comp
+L vitamins_included-rescue:GND-RESCUE-lets_split_panel-lets_split_panel-rescue #PWR?
+U 1 1 5B621855
+P 5700 5550
+F 0 "#PWR?" H 5700 5300 50  0001 C CNN
+F 1 "GND" H 5700 5400 50  0000 C CNN
+F 2 "" H 5700 5550 50  0000 C CNN
+F 3 "" H 5700 5550 50  0000 C CNN
+	1    5700 5550
+	1    0    0    -1
+$EndComp
 $EndSCHEMATC
