File: right.sch (KiCad schematic (older format))
At the start: 53 parts, among them J5 Speaker, J6 ISP, J8 WS2812>, P5 UJ2-MBH-1-SMT, P6 >WS2812, P8 SJ-43514-SMT, SW25 Socket, SW26 Socket, SW27 Socket, SW28 Socket, SW29 Socket, SW30 Socket, SW31 Socket, SW32 Socket, SW33 Socket, SW34 Socket, SW35 Socket, SW36 Socket, SW37 Socket, SW38 Socket, SW39 Socket, SW40 Socket, SW41 Socket, SW42 Socket, SW43 Socket, SW44 Socket, SW45 Socket, SW46 Socket, SW47 Socket, SW48 Socket, U2 ATMega32U4, Y2 16MHz

Commit message: renamed files, and generated xy files
Parts:
- SW43: value Socket -> Socket-overlap
Changed lines of the file:
@@
 P 6250 5175
 F 0 "SW43" H 6250 5460 50  0000 C CNN
-F 1 "Socket" H 6250 5369 50  0000 C CNN
+F 1 "Socket-overlap" H 6250 5369 50  0000 C CNN
 F 2 "CherryMX:Kailh-socket" H 6250 5375 50  0001 C CNN
 F 3 "" H 6250 5375 50  0001 C CNN
@@
 	2100 4525 2625 4525
 $Comp
-L lets_split_panel-rescue:VCC-RESCUE-lets_split_panel #PWR?
+L lets_split_panel-rescue:VCC-RESCUE-lets_split_panel #PWR010
 U 1 1 5B5311D3
 P 2175 6925
-F 0 "#PWR?" H 2175 6775 50  0001 C CNN
+F 0 "#PWR010" H 2175 6775 50  0001 C CNN
 F 1 "VCC" H 2175 7075 50  0000 C CNN
 F 2 "" H 2175 6925 50  0000 C CNN

Commit message: Added BOM and 3D file
Parts:
- C5, C6, C7, C8: symbol lets_split_panel-rescue:C_Small-RESCUE-lets_split_panel -> vitamins_included-rescue:C_Small-RESCUE-lets_split_panel-lets_split_panel-rescue
- J5: symbol lets_split_panel-rescue:Conn_01x02-RESCUE-lets_split_panel -> vitamins_included-rescue:Conn_01x02-RESCUE-lets_split_panel-lets_split_panel-rescue
- J6: symbol lets_split_panel-rescue:Conn_02x03_Odd_Even-RESCUE-lets_split_panel -> vitamins_included-rescue:Conn_02x03_Odd_Even-RESCUE-lets_split_panel-lets_split_panel-rescue
- J8: symbol lets_split_panel-rescue:Conn_01x01-RESCUE-lets_split_panel -> vitamins_included-rescue:Conn_01x01-RESCUE-lets_split_panel-lets_split_panel-rescue
- P5: symbol lets_split_panel-rescue:USB_OTG-RESCUE-lets_split-RESCUE-lets_split_panel -> vitamins_included-rescue:USB_OTG-RESCUE-lets_split-RESCUE-lets_split_panel-lets_split_panel-rescue
- P6: symbol lets_split_panel-rescue:Conn_01x03-RESCUE-lets_split_panel -> vitamins_included-rescue:Conn_01x03-RESCUE-lets_split_panel-lets_split_panel-rescue
- P8: symbol lets_split_panel-rescue:Conn_01x04-RESCUE-lets_split_panel -> vitamins_included-rescue:Conn_01x04-RESCUE-lets_split_panel-lets_split_panel-rescue
- R10, R7, R8, R9: symbol lets_split_panel-rescue:R_Small-RESCUE-lets_split_panel -> vitamins_included-rescue:R_Small-RESCUE-lets_split_panel-lets_split_panel-rescue
- SW25, SW26, SW27, SW28, SW29, SW30, SW31, SW32, SW33, SW34, SW35, SW36, SW37, SW38, SW39, SW40, SW41, SW42, SW43, SW44, SW45, SW46, SW47, SW48: symbol lets_split_panel-rescue:SW_Push-RESCUE-lets_split_panel -> vitamins_included-rescue:SW_Push-RESCUE-lets_split_panel-lets_split_panel-rescue
- U2: symbol lets_split_panel-rescue:ATMega32U4-RESCUE-lets_split_panel -> vitamins_included-rescue:ATMega32U4-RESCUE-lets_split_panel-lets_split_panel-rescue
- Y2: symbol lets_split_panel-rescue:Crystal-RESCUE-lets_split_panel -> vitamins_included-rescue:Crystal-RESCUE-lets_split_panel-lets_split_panel-rescue

Commit message: Added resistors to allow MCU to determin which half it is on
Parts:
- added J4: reset, Connector_PinHeader_2.54mm:PinHeader_1x02_P2.54mm_Vertical, symbol Connector_Generic:Conn_01x02
- added R12: 4k7, Resistor_SMD:R_0603_1608Metric, symbol vitamins_included-rescue:R_Small-RESCUE-lets_split_panel-lets_split_panel-rescue
- R10, R7, R8, R9: footprint Resistors_SMD:R_0603 -> Resistor_SMD:R_0603_1608Metric
- SW25, SW26, SW27, SW28, SW29, SW30, SW31, SW32, SW33, SW34, SW35, SW36, SW37, SW38, SW39, SW40, SW41, SW42, SW43, SW44, SW45, SW46, SW47, SW48: footprint CherryMX:Kailh-socket -> sockets:Kailh-socket
Connections:
- wire segments 150 -> 155

Commit message: Changed to USB-C connector
Parts:
- removed P5: UJ2-MBH-1-SMT, Connectors:USB-Mini-B-SMD, symbol vitamins_included-rescue:USB_OTG-RESCUE-lets_split-RESCUE-lets_split_panel-lets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
- added J10: 12401598E4#2A, Connector_USB:USB_C_Receptacle_Amphenol_12401610E4-2A, symbol Connector:USB_C_Receptacle
Connections:
- wire segments 155 -> 172

Commit message: Added resistors to allow the firmware to determine version
Parts:
- added R14: 4k7, Resistor_SMD:R_0603_1608Metric, symbol vitamins_included-rescue:R_Small-RESCUE-lets_split_panel-lets_split_panel-rescue
- SW43: value Socket-overlap -> Socket
Connections:
- wire segments 172 -> 175
Changed lines of the file:
@@
 P 6250 3000
 F 0 "SW43" H 6250 3285 50  0000 C CNN
-F 1 "Socket-overlap" H 6250 3194 50  0000 C CNN
+F 1 "Socket" H 6250 3194 50  0000 C CNN
 F 2 "sockets:Kailh-socket" H 6250 3200 50  0001 C CNN
 F 3 "" H 6250 3200 50  0001 C CNN
@@
 Wire Wire Line
 	1225 7200 1325 7200
+$Comp
+L vitamins_included-rescue:R_Small-RESCUE-lets_split_panel-lets_split_panel-rescue R14
+U 1 1 5B5A095B
+P 5425 4550
+F 0 "R14" H 5275 4575 50  0000 L CNN
+F 1 "4k7" H 5250 4500 50  0000 L CNN
+F 2 "Resistor_SMD:R_0603_1608Metric" H 5425 4550 50  0001 C CNN
+F 3 "" H 5425 4550 50  0000 C CNN
+	1    5425 4550
+	0    -1   -1   0
+$EndComp
+Wire Wire Line
+	5100 4550 5325 4550
+Wire Wire Line
+	5525 4550 5575 4550
+Wire Wire Line
+	5575 4550 5575 4600
+$Comp
+L power:GND #PWR033
+U 1 1 5B5B9F91
+P 5575 4600
+F 0 "#PWR033" H 5575 4350 50  0001 C CNN
+F 1 "GND" H 5580 4427 50  0000 C CNN
+F 2 "" H 5575 4600 50  0001 C CNN
+F 3 "" H 5575 4600 50  0001 C CNN
+	1    5575 4600
+	1    0    0    -1
+$EndComp
 $EndSCHEMATC

Commit message: changed to rounded passive footprints
Parts:
- C5, C6, C7, C8: footprint Capacitors_SMD:C_0603 -> Capacitor_SMD:C_0603_1608Metric
- R10: value 200R -> 220R
- R12, R14: value 4k7 -> 220R
Changed lines of the file:
@@
 P 2925 1050
 F 0 "R10" H 2955 1070 50  0000 L CNN
-F 1 "200R" H 2955 1010 50  0000 L CNN
+F 1 "220R" H 2955 1010 50  0000 L CNN
 F 2 "Resistor_SMD:R_0603_1608Metric" H 2925 1050 50  0001 C CNN
 F 3 "" H 2925 1050 50  0000 C CNN
@@
 F 0 "C8" H 3442 6246 50  0000 L CNN
 F 1 "1uF" H 3442 6155 50  0000 L CNN
-F 2 "Capacitors_SMD:C_0603" H 3350 6200 50  0001 C CNN
+F 2 "Capacitor_SMD:C_0603_1608Metric" H 3350 6200 50  0001 C CNN
 F 3 "" H 3350 6200 50  0001 C CNN
 	1    3350 6200
@@
 F 0 "C6" V 3175 5550 50  0000 C CNN
 F 1 "18pF" V 3150 5350 50  0000 C CNN
-F 2 "Capacitors_SMD:C_0603" H 3250 5450 50  0001 C CNN
+F 2 "Capacitor_SMD:C_0603_1608Metric" H 3250 5450 50  0001 C CNN
 F 3 "" H 3250 5450 50  0001 C CNN
 	1    3250 5450
@@
 F 0 "C7" V 3425 5850 50  0000 C CNN
 F 1 "18pF" V 3350 5850 50  0000 C CNN
-F 2 "Capacitors_SMD:C_0603" H 3250 5850 50  0001 C CNN
+F 2 "Capacitor_SMD:C_0603_1608Metric" H 3250 5850 50  0001 C CNN
 F 3 "" H 3250 5850 50  0001 C CNN
 	1    3250 5850
@@
 F 0 "C5" H 3142 6796 50  0000 L CNN
 F 1 "1uF" H 3142 6705 50  0000 L CNN
-F 2 "Capacitors_SMD:C_0603" H 3050 6750 50  0001 C CNN
+F 2 "Capacitor_SMD:C_0603_1608Metric" H 3050 6750 50  0001 C CNN
 F 3 "" H 3050 6750 50  0001 C CNN
 	1    3050 6750
@@
 P 5425 4450
 F 0 "R12" H 5455 4470 50  0000 L CNN
-F 1 "4k7" H 5455 4410 50  0000 L CNN
+F 1 "220R" H 5455 4410 50  0000 L CNN
 F 2 "Resistor_SMD:R_0603_1608Metric" H 5425 4450 50  0001 C CNN
 F 3 "" H 5425 4450 50  0000 C CNN
@@
 U 1 1 5B5A095B
 P 5425 4550
-F 0 "R14" H 5275 4575 50  0000 L CNN
-F 1 "4k7" H 5250 4500 50  0000 L CNN
+F 0 "R14" H 5250 4575 50  0000 L CNN
+F 1 "220R" H 5200 4500 50  0000 L CNN
 F 2 "Resistor_SMD:R_0603_1608Metric" H 5425 4550 50  0001 C CNN
 F 3 "" H 5425 4550 50  0000 C CNN

Commit message: Switched to connectors
Parts:
- J10: value 12401598E4#2A -> UTC16-G; footprint Connector_USB:USB_C_Receptacle_Amphenol_12401610E4-2A -> Connector_USB:USB_C_Receptacle_Palconn_UTC16-G
- J8: value WS2812> -> Sig
- P6: value >WS2812 -> WS2812
Changed lines of the file:
@@
 P 1525 1125
 F 0 "P6" H 1525 1325 50  0000 C CNN
-F 1 ">WS2812" V 1625 1125 50  0000 C CNN
+F 1 "WS2812" V 1625 1125 50  0000 C CNN
 F 2 "Wirepads:SMD_PAD_1x03_Pitch2.54mm" H 1525 1125 50  0001 C CNN
 F 3 "" H 1525 1125 50  0000 C CNN
@@
 P 1875 1125
 F 0 "J8" H 1795 900 50  0000 C CNN
-F 1 "WS2812>" H 1795 991 50  0000 C CNN
+F 1 "Sig" H 1795 991 50  0000 C CNN
 F 2 "Pin_Headers:Pin_Header_Straight_1x01_Pitch2.54mm" H 1875 1125 50  0001 C CNN
 F 3 "~" H 1875 1125 50  0001 C CNN
@@
 P 1425 5550
 F 0 "J10" H 1530 7117 50  0000 C CNN
-F 1 " 12401598E4#2A " H 1530 7026 50  0000 C CNN
-F 2 "Connector_USB:USB_C_Receptacle_Amphenol_12401610E4-2A" H 1575 5550 50  0001 C CNN
+F 1 "UTC16-G" H 1530 7026 50  0000 C CNN
+F 2 "Connector_USB:USB_C_Receptacle_Palconn_UTC16-G" H 1575 5550 50  0001 C CNN
 F 3 "http://www.usb.org/developers/docs/usb_31_033017.zip" H 1575 5550 50  0001 C CNN
 	1    1425 5550

Commit message: Added reset button, led, 3D models
Parts:
- added D28: red, LED_SMD:LED_0603_1608Metric_Castellated, symbol Device:LED_Small
- added R16: 220R, Resistor_SMD:R_0603_1608Metric, symbol vitamins_included-rescue:R_Small-RESCUE-lets_split_panel-lets_split_panel-rescue
- added SW50: FSMSM, Button_Switch_SMD:SW_SPST_FSMSM, symbol Switch:SW_SPST
Connections:
- wire segments 175 -> 187
Changed lines of the file:
@@
 L vitamins_included-rescue:Conn_02x03_Odd_Even-RESCUE-lets_split_panel-lets_split_panel-rescue J6
 U 1 1 5A0E2A70
-P 10325 4125
-F 0 "J6" H 10375 4442 50  0000 C CNN
-F 1 "ISP" H 10375 4351 50  0000 C CNN
-F 2 "Connector:Tag-Connect_TC2030-IDC-NL_2x03_P1.27mm_Vertical" H 10325 4125 50  0001 C CNN
-F 3 "" H 10325 4125 50  0001 C CNN
-	1    10325 4125
-	1    0    0    -1
-$EndComp
-Text Label 10125 4225 2    55   ~ 0
+P 2950 2050
+F 0 "J6" H 3000 2367 50  0000 C CNN
+F 1 "ISP" H 3000 2276 50  0000 C CNN
+F 2 "Connector:Tag-Connect_TC2030-IDC-NL_2x03_P1.27mm_Vertical" H 2950 2050 50  0001 C CNN
+F 3 "" H 2950 2050 50  0001 C CNN
+	1    2950 2050
+	1    0    0    -1
+$EndComp
+Text Label 2750 2150 2    55   ~ 0
 ~RESET
-Text Label 10125 4125 2    55   ~ 0
+Text Label 2750 2050 2    55   ~ 0
 SCK
-Text Label 3375 4500 2    35   ~ 0
+Text Label 3250 4500 2    35   ~ 0
 ~RESET
 Text Label 5100 4250 0    55   ~ 0
@@
 SCK
 Wire Wire Line
-	10625 4225 10675 4225
-Wire Wire Line
-	10675 4225 10675 4275
-Wire Wire Line
-	10625 4025 10675 4025
-Wire Wire Line
-	10675 4025 10675 3975
+	3250 2150 3300 2150
+Wire Wire Line
+	3300 2150 3300 2200
+Wire Wire Line
+	3250 1950 3300 1950
+Wire Wire Line
+	3300 1950 3300 1900
 $Comp
 L vitamins_included-rescue:VCC-RESCUE-lets_split_panel-lets_split_panel-rescue #PWR037
 U 1 1 5A0E2A84
-P 10675 3975
-F 0 "#PWR037" H 10675 3825 50  0001 C CNN
-F 1 "VCC" H 10675 4125 50  0000 C CNN
-F 2 "" H 10675 3975 50  0000 C CNN
-F 3 "" H 10675 3975 50  0000 C CNN
-	1    10675 3975
+P 3300 1900
+F 0 "#PWR037" H 3300 1750 50  0001 C CNN
+F 1 "VCC" H 3300 2050 50  0000 C CNN
+F 2 "" H 3300 1900 50  0000 C CNN
+F 3 "" H 3300 1900 50  0000 C CNN
+	1    3300 1900
 	1    0    0    -1
 $EndComp
@@
 L vitamins_included-rescue:GND-RESCUE-lets_split_panel-lets_split_panel-rescue #PWR038
 U 1 1 5A0E2A8A
-P 10675 4275
-F 0 "#PWR038" H 10675 4025 50  0001 C CNN
-F 1 "GND" H 10675 4125 50  0000 C CNN
-F 2 "" H 10675 4275 50  0000 C CNN
-F 3 "" H 10675 4275 50  0000 C CNN
-	1    10675 4275
-	1    0    0    -1
-$EndComp
-Text Label 10125 4025 2    55   ~ 0
+P 3300 2200
+F 0 "#PWR038" H 3300 1950 50  0001 C CNN
+F 1 "GND" H 3300 2050 50  0000 C CNN
+F 2 "" H 3300 2200 50  0000 C CNN
+F 3 "" H 3300 2200 50  0000 C CNN
+	1    3300 2200
+	1    0    0    -1
+$EndComp
+Text Label 2750 1950 2    55   ~ 0
 MISO
-Text Label 10625 4125 0    55   ~ 0
+Text Label 3250 2050 0    55   ~ 0
 MOSI
 Text Label 2325 5150 0    60   ~ 0
@@
 L Connector_Generic:Conn_01x02 J4
 U 1 1 5B54699A
-P 2525 4500
-F 0 "J4" H 2605 4492 50  0000 L CNN
-F 1 "reset" H 2605 4401 50  0000 L CNN
-F 2 "Connector_PinHeader_2.54mm:PinHeader_1x02_P2.54mm_Vertical" H 2525 4500 50  0001 C CNN
-F 3 "~" H 2525 4500 50  0001 C CNN
-	1    2525 4500
+P 1300 1975
+F 0 "J4" H 1380 1967 50  0000 L CNN
+F 1 "reset" H 1380 1876 50  0000 L CNN
+F 2 "Connector_PinHeader_2.54mm:PinHeader_1x02_P2.54mm_Vertical" H 1300 1975 50  0001 C CNN
+F 3 "~" H 1300 1975 50  0001 C CNN
+	1    1300 1975
 	-1   0    0    -1
-$EndComp
-Wire Wire Line
-	2725 4500 2850 4500
-Connection ~ 2850 4500
-Wire Wire Line
-	2725 4600 2800 4600
-Wire Wire Line
-	2800 4600 2800 4650
-$Comp
-L vitamins_included-rescue:GND-RESCUE-lets_split_panel-lets_split_panel-rescue #PWR016
-U 1 1 5B56EBA6
-P 2800 4650
-F 0 "#PWR016" H 2800 4400 50  0001 C CNN
-F 1 "GND" H 2800 4500 50  0000 C CNN
-F 2 "" H 2800 4650 50  0000 C CNN
-F 3 "" H 2800 4650 50  0000 C CNN
-	1    2800 4650
-	1    0    0    -1
 $EndComp
 Wire Wire Line
@@
 	1    0    0    -1
 $EndComp
+$Comp
+L vitamins_included-rescue:GND-RESCUE-lets_split_panel-lets_split_panel-rescue #PWR016
+U 1 1 5B62A621
+P 1550 2325
+F 0 "#PWR016" H 1550 2075 50  0001 C CNN
+F 1 "GND" H 1550 2175 50  0000 C CNN
+F 2 "" H 1550 2325 50  0000 C CNN
+F 3 "" H 1550 2325 50  0000 C CNN
+	1    1550 2325
+	1    0    0    -1
+$EndComp
+$Comp
+L Switch:SW_SPST SW50
+U 1 1 5B62A627
+P 1600 2025
+F 0 "SW50" V 1554 2123 50  0000 L CNN
+F 1 "FSMSM" V 1645 2123 50  0000 L CNN
+F 2 "Button_Switch_SMD:SW_SPST_FSMSM" H 1600 2025 50  0001 C CNN
+F 3 "" H 1600 2025 50  0001 C CNN
+	1    1600 2025
+	0    1    1    0
+$EndComp
+Wire Wire Line
+	1500 1975 1550 1975
+Wire Wire Line
+	1550 1975 1550 1775
+Wire Wire Line
+	1550 1775 1600 1775
+Wire Wire Line
+	1600 1775 1600 1825
+Wire Wire Line
+	1500 2075 1550 2075
+Wire Wire Line
+	1550 2275 1600 2275
+Wire Wire Line
+	1600 2275 1600 2225
+Wire Wire Line
+	1550 2075 1550 2275
+Connection ~ 1550 2275
+Wire Wire Line
+	1550 2275 1550 2325
+Wire Wire Line
+	1550 1775 1550 1700
+Connection ~ 1550 1775
+Text Label 1550 1700 3    35   ~ 0
+~RESET
+$Comp
+L Device:LED_Small D28
+U 1 1 5B5FD568
+P 5300 5550
+F 0 "D28" H 5300 5345 50  0000 C CNN
+F 1 "red" H 5300 5436 50  0000 C CNN
+F 2 "LED_SMD:LED_0603_1608Metric_Castellated" V 5300 5550 50  0001 C CNN
+F 3 "~" V 5300 5550 50  0001 C CNN
+	1    5300 5550
+	-1   0    0    1
+$EndComp
+Wire Wire Line
+	5175 5650 5175 5550
+Wire Wire Line
+	5175 5550 5200 5550
+$Comp
+L vitamins_included-rescue:R_Small-RESCUE-lets_split_panel-lets_split_panel-rescue R16
+U 1 1 5B5FD571
+P 5500 5550
+F 0 "R16" H 5525 5575 50  0000 L CNN
+F 1 "220R" H 5525 5500 50  0000 L CNN
+F 2 "Resistor_SMD:R_0603_1608Metric" H 5500 5550 50  0001 C CNN
+F 3 "" H 5500 5550 50  0000 C CNN
+	1    5500 5550
+	0    -1   -1   0
+$EndComp
+Wire Wire Line
+	5175 5650 5100 5650
+$Comp
+L power:GND #PWR?
+U 1 1 5B5E458B
+P 5650 5600
+F 0 "#PWR?" H 5650 5350 50  0001 C CNN
+F 1 "GND" H 5655 5427 50  0000 C CNN
+F 2 "" H 5650 5600 50  0001 C CNN
+F 3 "" H 5650 5600 50  0001 C CNN
+	1    5650 5600
+	1    0    0    -1
+$EndComp
+Wire Wire Line
+	5600 5550 5650 5550
+Wire Wire Line
+	5650 5550 5650 5600
 $EndSCHEMATC
